Commit message: 7 dof kinodynamic and constraint fixings

File: iiwa_cup.urdf (robot description, URDF)
Before this commit: robot iiwa, 11 links, 10 joints
Joints:
- joint F_joint_cup: origin xyz=0 0 0.1 rpy=0 0 0 -> xyz=0 0 0.1 rpy=-1.57 0 0

Commit message: 16kg of mass and colors added

File: iiwa_cup.urdf (robot description, URDF)
Before this commit: robot iiwa, 11 links, 10 joints
Links:
- link F_link_cup: mass 8.0 -> 16.0

Commit message: change to 12kg

File: iiwa_cup.urdf (robot description, URDF)
Before this commit: robot iiwa, 11 links, 10 joints
Links:
- link F_link_cup: mass 16.0 -> 12.0

Commit message: Cuboid 14kg

File: iiwa_cup.urdf (robot description, URDF)
Before this commit: robot iiwa, 11 links, 10 joints
Links:
- link F_link_cup: mass 12.0 -> 14.0

Commit message: Updated version of the collsion loss

File: iiwa_cup.urdf (robot description, URDF)
Before this commit: robot iiwa, 11 links, 10 joints
Links:
- link F_link_cup: mass 14.0 -> 12.0; geometry visual box size=0.2 0.2 0.3
