Commit message: release of the manifold planning

File: iiwa_striker.urdf (robot description, URDF)
Before this commit: robot iiwa_striker, 14 links, 13 joints
Links:
- removed link F_striker_base
- removed link front_base
- added link F_striker_tip, mass 0.350; collision mesh filename=./meshes_new/striker/collision/EE_arm_collision.stl; visual mesh filename=./meshes_new/striker/visual/EE_arm.stl
- added link world
- link F_link_0: mass 5 -> 5.476713; geometry collision mesh filename=./meshes_new/iiwa/collision/link_0.stl; visual mesh filename=./meshes_new/iiwa/visual/link_0.stl
- link F_link_1: mass 3.947808 -> 4.100238; geometry collision mesh filename=./meshes_new/iiwa/collision/link_1.stl; visual mesh filename=./meshes_new/iiwa/visual/link_1.stl
- link F_link_2: mass 4.502752 -> 3.943457; geometry collision mesh filename=./meshes_new/iiwa/collision/link_2.stl; visual mesh filename=./meshes_new/iiwa/visual/link_2.stl
- link F_link_3: mass 2.455197 -> 4; geometry collision mesh filename=./meshes_new/iiwa/collision/link_3.stl; visual mesh filename=./meshes_new/iiwa/visual/link_3.stl
- link F_link_4: mass 2.611550 -> 4; geometry collision mesh filename=./meshes_new/iiwa/collision/link_4.stl; visual mesh filename=./meshes_new/iiwa/visual/link_4.stl
- link F_link_5: mass 3.410009 -> 3.2; geometry collision mesh filename=./meshes_new/iiwa/collision/link_5.stl; visual mesh filename=./meshes_new/iiwa/visual/link_5.stl
- link F_link_6: mass 3.387949 -> 2.2; geometry collision mesh filename=./meshes_new/iiwa/collision/link_6.stl; visual mesh filename=./meshes_new/iiwa/visual/link_6.stl
- link F_link_7: mass 0.354321 -> 0.4; geometry collision mesh filename=./meshes_new/iiwa/collision/link_7.stl; visual mesh filename=./meshes_new/iiwa/visual/link_7.stl
- link F_striker_joint_link: mass 0.01 -> 0.05
- link F_striker_mallet: geometry collision cylinder length=0.04 radius=0.04815; visual mesh filename=./meshes_new/striker/visual/EE_mallet_foam.stl
- link F_striker_mallet_tip: mass 0.1 -> 0.05
Joints:
- removed joint front_base_F_base_joint
- added joint world_F_base_joint: type fixed, parent world, child F_link_0, origin xyz=0 0 0 rpy=0 0 0
- joint F_joint_ee: axis 0 0 1 -> (none)
- joint F_striker: child F_striker_base -> F_striker_tip; origin xyz=0.0 0.0 0.0 rpy=0 0 0 -> xyz=0.0 0.0 0.515 rpy=0 0 0
- joint F_striker_joint_1: limit lower=-1.5707963267948966 upper=1.5707963267948966 effort=1 velocity=100 -> lower=-1.5707963267948966 upper=1.5707963267948966 effort=1 velocity=3.1415926; origin xyz=0.0 0.0 0.515 rpy=0 0 0 -> xyz=0.0 0.0 0.0 rpy=0 0 0; parent F_striker_base -> F_striker_tip
- joint F_striker_joint_2: limit lower=-1.5707963267948966 upper=1.5707963267948966 effort=1 velocity=100 -> lower=-1.5707963267948966 upper=1.5707963267948966 effort=1 velocity=3.1415926
- joint F_striker_mallet_fix: origin xyz=0.0 0.0 0.095 rpy=0 0 0 -> xyz=0.0 0.0 0.0645 rpy=0 0 0
